File: PCB/rx.brd (EAGLE design)
At the start: 97.8 x 64.8 mm, 8 parts

Commit message: PCB
Parts:
- U1: device SparkFun-IC-Power:SOT223 -> rx:SOT223
Routing:
- net +3.3V: track 56.9 -> 36.6 mm
- net D7: track 27.5 -> 39.6 mm
- net GND: track 206.7 -> 208.5 mm
- net D12: track 39.2 -> 40.0 mm
- net D13: track 65.7 -> 66.3 mm, vias 1 -> 0
