File: PCB/rx.sch (EAGLE design)
At the start: 8 parts

Commit message: PCB
Parts:
- U1: device SparkFun-IC-Power:V_REG_LM1117SOT223 -> rx:V_REG_LM1117SOT223
Changed lines of the file:
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@@
 <part name="ESP" library="rx" deviceset="ESP8266_MODULE" device=""/>
 <part name="NRF" library="rx" deviceset="NRF24L01_MODULE" device="_PA"/>
-<part name="U1" library="SparkFun-IC-Power" deviceset="V_REG_LM1117" device="SOT223"/>
 <part name="FRAME1" library="frames" deviceset="LETTER_L" device=""/>
 <part name="POWER" library="rx" deviceset="POWER_REDUCE" device=""/>
@@
 <part name="RELAY" library="rx" deviceset="RELAY_MODULE" device=""/>
 <part name="BUZZ" library="rx" deviceset="BUZZ_MODULE" device=""/>
+<part name="U1" library="rx" deviceset="V_REG_LM1117" device="SOT223"/>
 </parts>
 <sheets>
@@
 <instance part="ESP" gate="G$1" x="104.14" y="756.92"/>
 <instance part="NRF" gate="G$1" x="104.14" y="777.24"/>
-<instance part="U1" gate="G$1" x="111.76" y="833.12"/>
 <instance part="FRAME1" gate="G$1" x="30.48" y="657.86"/>
 <instance part="FRAME1" gate="G$2" x="177.8" y="657.86"/>
@@
 <instance part="RELAY" gate="G$1" x="119.38" y="805.18" rot="R180"/>
 <instance part="BUZZ" gate="G$1" x="73.66" y="784.86"/>
+<instance part="U1" gate="G$1" x="111.76" y="833.12"/>
 </instances>
 <busses>
@@
 </segment>
 <segment>
-<pinref part="U1" gate="G$1" pin="IN"/>
 <wire x1="104.14" y1="833.12" x2="101.6" y2="833.12" width="0.1524" layer="91"/>
 <label x="101.6" y="833.12" size="1.778" layer="95"/>
+<pinref part="U1" gate="G$1" pin="IN"/>
 </segment>
 <segment>
@@
 </segment>
 <segment>
-<pinref part="U1" gate="G$1" pin="ADJ"/>
 <wire x1="111.76" y1="825.5" x2="111.76" y2="822.96" width="0.1524" layer="91"/>
 <label x="109.22" y="822.96" size="1.778" layer="95"/>
+<pinref part="U1" gate="G$1" pin="ADJ"/>
 </segment>
 <segment>
@@
 <net name="+3.3V" class="0">
 <segment>
-<pinref part="U1" gate="G$1" pin="OUT@1"/>
 <wire x1="119.38" y1="830.58" x2="121.92" y2="830.58" width="0.1524" layer="91"/>
 <label x="119.38" y="830.58" size="1.778" layer="95"/>
+<pinref part="U1" gate="G$1" pin="OUT@1"/>
 </segment>
 <segment>
-<pinref part="U1" gate="G$1" pin="OUT"/>
 <wire x1="119.38" y1="833.12" x2="121.92" y2="833.12" width="0.1524" layer="91"/>
 <label x="119.38" y="833.12" size="1.778" layer="95"/>
+<pinref part="U1" gate="G$1" pin="OUT"/>
 </segment>
 <segment>
