File: PCB/tag_key.sch (EAGLE design)
At the start: 7 parts

Commit message: tag,mail
Parts:
- removed SW1: (no value), tag_key:SEEED-OPL-SWITCH_SMD-BUTTON(4P-6.0X6.0X7.5MM)
- added SW3: (no value), tag_key:SEEED-OPL-SWITCH_SMD-BUTTON(4P-6.0X6.0X3LEGM)
Connections:
- net N$2: now also SW3.A1; no longer SW1.A1
- net P1.6: now also SW3.B1; no longer SW1.B1
Changed lines of the file:
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@@
 <part name="FRAME1" library="tag_key" deviceset="RX_LETTER_L" device=""/>
 <part name="BAT1" library="tag_key" deviceset="SEEED-OPL-CONNECTOR_DIP-BATTERY-CELL-HOLDER(2032)" device="" value="cr2032"/>
-<part name="SW1" library="tag_key" deviceset="SEEED-OPL-SWITCH_SMD-BUTTON(4P-6.0X6.0X7.5MM)" device=""/>
 <part name="SW2" library="tag_key" deviceset="SEEED-OPL-SWITCH_SMD-BUTTON(4P-6.0X6.0X7.5MM)" device=""/>
 <part name="J1" library="tag_key" deviceset="SPARKFUN-CONNECTORS_CONN_08" device="&quot;"/>
 <part name="J2" library="tag_key" deviceset="SPARKFUN-CONNECTORS_CONN_11" device="_1.27MM"/>
+<part name="SW3" library="tag_key" deviceset="SEEED-OPL-SWITCH_SMD-BUTTON(4P-6.0X6.0X3LEGM)" device=""/>
 </parts>
 <sheets>
@@
 <instance part="FRAME1" gate="G$2" x="142.24" y="-2.54"/>
 <instance part="BAT1" gate="G$1" x="81.28" y="154.94"/>
-<instance part="SW1" gate="G$1" x="35.56" y="160.02"/>
 <instance part="SW2" gate="G$1" x="35.56" y="147.32"/>
 <instance part="J1" gate="G$1" x="78.74" y="121.92"/>
 <instance part="J2" gate="G$1" x="30.48" y="121.92"/>
+<instance part="SW3" gate="G$1" x="35.56" y="160.02"/>
 </instances>
 <busses>
@@
 </segment>
 <segment>
-<pinref part="SW1" gate="G$1" pin="B1"/>
+<pinref part="SW3" gate="G$1" pin="B1"/>
 <wire x1="44.45" y1="157.48" x2="54.61" y2="157.48" width="0.1524" layer="91"/>
-<label x="46.99" y="157.48" size="1.778" layer="95"/>
+<label x="48.26" y="157.48" size="1.778" layer="95"/>
 </segment>
 </net>
@@
 <wire x1="21.59" y1="162.56" x2="21.59" y2="167.64" width="0.1524" layer="91"/>
 <wire x1="21.59" y1="167.64" x2="44.45" y2="167.64" width="0.1524" layer="91"/>
-<pinref part="SW1" gate="G$1" pin="A1"/>
+<pinref part="SW3" gate="G$1" pin="A1"/>
 <wire x1="44.45" y1="167.64" x2="44.45" y2="162.56" width="0.1524" layer="91"/>
 </segment>
