File: PCB/tag_key-v1.brd (EAGLE design)
At the start: 44.5 x 29 mm, 7 parts

Commit message: new bike
Routing:
- net GND: track 0.00 -> 49.7 mm
- net +3.3: track 0.00 -> 29.4 mm
- net P1.5: track 0.00 -> 27.1 mm
- net RST: track 0.00 -> 25.5 mm
- net P1.1: track 0.25 -> 21.1 mm
- net P1.0: track 0.00 -> 17.9 mm
- net P1.6: track 0.00 -> 15.7 mm
- net P0.7: track 0.22 -> 15.0 mm
- net N$2: track 0.00 -> 13.1 mm
- net P0.5: track 0.00 -> 11.2 mm
- net PROG: track 0.00 -> 9.35 mm
- net N$1: track 0.00 -> 7.26 mm
