File: PCB/room/untitled.brd (EAGLE design)
At the start: 63 x 66 mm, 5 parts

Commit message: auto_door
Parts:
- added J1: (no value), rx:2.54*4
Connections:
- net N$16 renamed RX
- net +5V: now also J1.4
- net D1: now also RX.3
- net D2: now also RELAY.3; no longer RX.3
- net D3: now also RELAY.4; no longer RELAY.3
- net D4: no longer RELAY.4
- net GND: now also J1.1, J1.2, J1.3
Changed lines of the file:
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@@
 <setting verticaltext="up"/>
 </settings>
-<grid distance="1" unitdist="mm" unit="mm" style="lines" multiple="1" display="yes" altdistance="1" altunitdist="mm" altunit="mm"/>
+<grid distance="0.1" unitdist="mm" unit="mm" style="lines" multiple="1" display="yes" altdistance="1" altunitdist="mm" altunit="mm"/>
 <layers>
 <layer number="1" name="Top" color="4" fill="1" visible="yes" active="yes"/>
@@
 <param name="mtCopper" value="0.035mm 0.035mm 0.035mm 0.035mm 0.035mm 0.035mm 0.035mm 0.035mm 0.035mm 0.035mm 0.035mm 0.035mm 0.035mm 0.035mm 0.035mm 0.035mm"/>
 <param name="mtIsolate" value="1.5mm 0.15mm 0.2mm 0.15mm 0.2mm 0.15mm 0.2mm 0.15mm 0.2mm 0.15mm 0.2mm 0.15mm 0.2mm 0.15mm 0.2mm"/>
-<param name="mdWireWire" value="30mil"/>
-<param name="mdWirePad" value="30mil"/>
-<param name="mdWireVia" value="30mil"/>
-<param name="mdPadPad" value="30mil"/>
-<param name="mdPadVia" value="30mil"/>
-<param name="mdViaVia" value="30mil"/>
-<param name="mdSmdPad" value="30mil"/>
-<param name="mdSmdVia" value="30mil"/>
-<param name="mdSmdSmd" value="30mil"/>
+<param name="mdWireWire" value="10mil"/>
+<param name="mdWirePad" value="10mil"/>
+<param name="mdWireVia" value="10mil"/>
+<param name="mdPadPad" value="10mil"/>
+<param name="mdPadVia" value="10mil"/>
+<param name="mdViaVia" value="10mil"/>
+<param name="mdSmdPad" value="10mil"/>
+<param name="mdSmdVia" value="10mil"/>
+<param name="mdSmdSmd" value="10mil"/>
 <param name="mdViaViaSameLayer" value="8mil"/>
 <param name="mnLayersViaInSmd" value="2"/>
@@
 <param name="mdDrill" value="8mil"/>
 <param name="mdSmdStop" value="0mil"/>
-<param name="msWidth" value="30mil"/>
+<param name="msWidth" value="10mil"/>
 <param name="msDrill" value="24mil"/>
 <param name="msMicroVia" value="9.99mm"/>
@@
 <param name="RoutingGrid" value="50mil"/>
 <param name="AutoGrid" value="1"/>
-<param name="Efforts" value="0"/>
+<param name="Efforts" value="2"/>
 <param name="TopRouterVariant" value="1"/>
 <param name="tpViaShape" value="round"/>
@@
 <element name="J" library="rx" package="OUT_HEAD_4_AC_2CH" value="" x="27" y="7" rot="R180"/>
 <element name="U" library="rx" package="ESP8266_MINI_SIDE" value="" x="11" y="48" rot="R270"/>
+<element name="J1" library="rx" package="2.54*4" value="" x="6" y="62" rot="R90"/>
 </elements>
 <signals>
@@
 <contactref element="RX" pad="4"/>
 <contactref element="U" pad="1"/>
+<contactref element="J1" pad="4"/>
 <wire x1="12.53" y1="58.61" x2="39.23" y2="61.32" width="0" layer="19" extent="1-1"/>
+<wire x1="3.97" y1="65.94" x2="12.53" y2="58.61" width="0" layer="19" extent="1-1"/>
 <wire x1="54.42" y1="30.31" x2="39.23" y2="61.32" width="0" layer="19" extent="1-1"/>
 <wire x1="12.32" y1="22.75" x2="12.53" y2="58.61" width="0" layer="19" extent="1-1"/>
@@
 <contactref element="RX" pad="1"/>
 <contactref element="U" pad="2"/>
+<contactref element="J1" pad="1"/>
+<contactref element="J1" pad="3"/>
+<contactref element="J1" pad="2"/>
 <wire x1="12.53" y1="56.07" x2="34.15" y2="61.32" width="0" layer="19" extent="1-1"/>
+<wire x1="3.97" y1="58.32" x2="12.53" y2="56.07" width="0" layer="19" extent="1-1"/>
+<wire x1="3.97" y1="60.86" x2="3.97" y2="58.32" width="0" layer="19" extent="1-1"/>
+<wire x1="3.97" y1="63.4" x2="3.97" y2="60.86" width="0" layer="19" extent="1-1"/>
 <wire x1="54.42" y1="35.39" x2="34.15" y2="61.32" width="0" layer="19" extent="1-1"/>
 <wire x1="12.32" y1="15.13" x2="12.53" y2="56.07" width="0" layer="19" extent="1-1"/>
@@
 <signal name="D1">
 <contactref element="U" pad="6"/>
+<contactref element="RX" pad="3"/>
+<wire x1="12.32" y1="20.21" x2="12.53" y2="45.91" width="0" layer="19" extent="1-1"/>
 </signal>
 <signal name="D2">
 <contactref element="U" pad="5"/>
-<contactref element="RX" pad="3"/>
-<wire x1="12.32" y1="20.21" x2="12.53" y2="48.45" width="0" layer="19" extent="1-1"/>
+<contactref element="RELAY" pad="3"/>
+<wire x1="12.53" y1="48.45" x2="29.07" y2="61.32" width="0" layer="19" extent="1-1"/>
 </signal>
 <signal name="D3">
 <contactref element="U" pad="4"/>
-<contactref element="RELAY" pad="3"/>
-<wire x1="12.53" y1="50.99" x2="29.07" y2="61.32" width="0" layer="19" extent="1-1"/>
+<contactref element="RELAY" pad="4"/>
+<wire x1="12.53" y1="50.99" x2="23.99" y2="61.32" width="0" layer="19" extent="1-1"/>
 </signal>
 <signal name="D4">
 <contactref element="U" pad="3"/>
-<contactref element="RELAY" pad="4"/>
-<wire x1="12.53" y1="53.53" x2="23.99" y2="61.32" width="0" layer="19" extent="1-1"/>
-</signal>
-<signal name="N$16">
-<contactref element="U" pad="7"/>
 </signal>
 <signal name="N$17">
 <contactref element="U" pad="8"/>
 </signal>
+<signal name="RX">
+<contactref element="U" pad="7"/>
+</signal>
 </signals>

Commit message: small_ac
Parts:
- added C1: (no value), resistor:E5-5
Connections:
- net +5V: now also C1.+
- net GND: now also C1.-
Routing:
- net +5V: track 0.00 -> 129.3 mm
- net GND: track 0.00 -> 124.5 mm
- net L: track 0.00 -> 31.1 mm
- net D1: track 0.00 -> 27.6 mm
- net D2: track 0.00 -> 22.0 mm
- net D3: track 0.00 -> 16.1 mm
- net OUT1: track 0.00 -> 15.6 mm
- net OUT2: track 0.00 -> 11.8 mm
- net N: track 0.00 -> 9.24 mm
