File: PCB/room/untitled.sch (EAGLE design)
At the start: 5 parts

Commit message: auto_door
Parts:
- added J1: (no value), rx:2.544
Connections:
- net N$16 renamed RX
- net +5V: now also J1.4
- net D1: now also RX.OUT
- net D2: now also RELAY.IN1; no longer RX.OUT
- net D3: now also RELAY.IN2; no longer RELAY.IN1
- net D4: no longer RELAY.IN2
- net GND: now also J1.1, J1.2, J1.3
Changed lines of the file:
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@@
 <part name="J" library="rx" deviceset="OUT_HEAD_4_AC_2CH" device=""/>
 <part name="U" library="rx" deviceset="ESP8266_MINI_SIDE" device=""/>
+<part name="J1" library="rx" deviceset="2.54*4" device=""/>
 </parts>
 <sheets>
@@
 <instance part="J" gate="G$1" x="71.12" y="63.5"/>
 <instance part="U" gate="G$1" x="66.04" y="-2.54"/>
+<instance part="J1" gate="G$1" x="99.06" y="-5.08" rot="R180"/>
 </instances>
 <busses>
@@
 <label x="78.74" y="2.54" size="1.778" layer="95"/>
 </segment>
+<segment>
+<pinref part="J1" gate="G$1" pin="4"/>
+<wire x1="96.52" y1="-2.54" x2="91.44" y2="-2.54" width="0.1524" layer="91"/>
+<label x="91.44" y="-2.54" size="1.778" layer="95"/>
+</segment>
 </net>
 <net name="GND" class="0">
@@
 <wire x1="76.2" y1="0" x2="83.82" y2="0" width="0.1524" layer="91"/>
 <label x="78.74" y="0" size="1.778" layer="95"/>
+</segment>
+<segment>
+<pinref part="J1" gate="G$1" pin="1"/>
+<wire x1="96.52" y1="-10.16" x2="91.44" y2="-10.16" width="0.1524" layer="91"/>
+<label x="91.44" y="-10.16" size="1.778" layer="95"/>
+</segment>
+<segment>
+<pinref part="J1" gate="G$1" pin="3"/>
+<wire x1="96.52" y1="-5.08" x2="91.44" y2="-5.08" width="0.1524" layer="91"/>
+<label x="91.44" y="-5.08" size="1.778" layer="95"/>
+</segment>
+<segment>
+<pinref part="J1" gate="G$1" pin="2"/>
+<wire x1="96.52" y1="-7.62" x2="91.44" y2="-7.62" width="0.1524" layer="91"/>
+<label x="91.44" y="-7.62" size="1.778" layer="95"/>
 </segment>
 </net>
@@
 <label x="78.74" y="-10.16" size="1.778" layer="95"/>
 </segment>
+<segment>
+<pinref part="RX" gate="G$1" pin="OUT"/>
+<wire x1="76.2" y1="15.24" x2="83.82" y2="15.24" width="0.1524" layer="91"/>
+<label x="78.74" y="15.24" size="1.778" layer="95"/>
+</segment>
 </net>
 <net name="D2" class="0">
@@
 </segment>
 <segment>
-<pinref part="RX" gate="G$1" pin="OUT"/>
-<wire x1="76.2" y1="15.24" x2="83.82" y2="15.24" width="0.1524" layer="91"/>
-<label x="78.74" y="15.24" size="1.778" layer="95"/>
+<pinref part="RELAY" gate="G$1" pin="IN1"/>
+<wire x1="76.2" y1="43.18" x2="83.82" y2="43.18" width="0.1524" layer="91"/>
+<label x="78.74" y="43.18" size="1.778" layer="95"/>
 </segment>
 </net>
@@
 </segment>
 <segment>
-<pinref part="RELAY" gate="G$1" pin="IN1"/>
-<wire x1="76.2" y1="43.18" x2="83.82" y2="43.18" width="0.1524" layer="91"/>
-<label x="78.74" y="43.18" size="1.778" layer="95"/>
+<pinref part="RELAY" gate="G$1" pin="IN2"/>
+<wire x1="76.2" y1="40.64" x2="83.82" y2="40.64" width="0.1524" layer="91"/>
+<label x="78.74" y="40.64" size="1.778" layer="95"/>
 </segment>
 </net>
@@
 <label x="78.74" y="-2.54" size="1.778" layer="95"/>
 </segment>
-<segment>
-<pinref part="RELAY" gate="G$1" pin="IN2"/>
-<wire x1="76.2" y1="40.64" x2="83.82" y2="40.64" width="0.1524" layer="91"/>
-<label x="78.74" y="40.64" size="1.778" layer="95"/>
-</segment>
-</net>
-<net name="N$16" class="0">
-<segment>
-<pinref part="U" gate="G$1" pin="RX"/>
-<wire x1="76.2" y1="-12.7" x2="83.82" y2="-12.7" width="0.1524" layer="91"/>
-</segment>
 </net>
 <net name="N$17" class="0">
@@
 </segment>
 </net>
+<net name="RX" class="0">
+<segment>
+<pinref part="U" gate="G$1" pin="RX"/>
+<wire x1="76.2" y1="-12.7" x2="83.82" y2="-12.7" width="0.1524" layer="91"/>
+<label x="78.74" y="-12.7" size="1.778" layer="95"/>
+</segment>
+</net>

Commit message: small_ac
Parts:
- added C1: (no value), resistor:CPOL-EUE5-5
Connections:
- net +5V: now also C1.+
- net GND: now also C1.-
Changed lines of the file:
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@@
 <part name="U" library="rx" deviceset="ESP8266_MINI_SIDE" device=""/>
 <part name="J1" library="rx" deviceset="2.54*4" device=""/>
+<part name="C1" library="resistor" deviceset="CPOL-EU" device="E5-5"/>
 </parts>
 <sheets>
@@
 <instance part="U" gate="G$1" x="66.04" y="-2.54"/>
 <instance part="J1" gate="G$1" x="99.06" y="-5.08" rot="R180"/>
+<instance part="C1" gate="G$1" x="104.14" y="17.78"/>
 </instances>
 <busses>
@@
 <label x="91.44" y="-2.54" size="1.778" layer="95"/>
 </segment>
+<segment>
+<pinref part="C1" gate="G$1" pin="+"/>
+<wire x1="104.14" y1="20.32" x2="96.52" y2="20.32" width="0.1524" layer="91"/>
+<label x="96.52" y="20.32" size="1.778" layer="95"/>
+</segment>
 </net>
 <net name="GND" class="0">
@@
 <label x="91.44" y="-7.62" size="1.778" layer="95"/>
 </segment>
+<segment>
+<pinref part="C1" gate="G$1" pin="-"/>
+<wire x1="104.14" y1="12.7" x2="96.52" y2="12.7" width="0.1524" layer="91"/>
+<label x="96.52" y="12.7" size="1.778" layer="95"/>
+</segment>
 </net>
